File: led_50w/led_50w.kicad_sch (KiCad schematic)
At the start: 49 parts

Commit message: rev 2 eeschema&layout
Parts:
- LED15: renamed from LED?; value (none) -> JB2835BWT-G-H40EA0000-N0000001; footprint (none) -> 2835-library:JB2835BWTGH40EA0000N0000001
- gave numbers to parts that had none: 48

Commit message: REV3-F
Parts:
- added TP1: TestPoint, symbol Connector:TestPoint
- added TP2: (no value), symbol Connector:TestPoint
Connections:
- net +24V: now also TP2.1
- net GND: now also TP1.1
Changed lines of the file:
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@@
   (junction (at 182.88 176.53) (diameter 0) (color 0 0 0 0)
   )
+  (junction (at 303.53 90.17) (diameter 0) (color 0 0 0 0)
+  )
   (junction (at 288.29 176.53) (diameter 0) (color 0 0 0 0)
   )
@@
   (junction (at 207.01 162.56) (diameter 0) (color 0 0 0 0)
   )
+  (junction (at 288.29 200.66) (diameter 0) (color 0 0 0 0)
+  )
   (junction (at 62.23 125.73) (diameter 0) (color 0 0 0 0)
   )
@@
     (stroke (width 0) (type default) (color 0 0 0 0))
   )
-  (wire (pts (xy 303.53 86.36) (xy 303.53 111.76))
+  (wire (pts (xy 303.53 86.36) (xy 303.53 90.17))
     (stroke (width 0) (type default) (color 0 0 0 0))
   )
@@
     (stroke (width 0) (type default) (color 0 0 0 0))
   )
+  (wire (pts (xy 303.53 90.17) (xy 327.66 90.17))
+    (stroke (width 0) (type default) (color 0 0 0 0))
+  )
   (wire (pts (xy 247.65 176.53) (xy 247.65 189.23))
     (stroke (width 0) (type default) (color 0 0 0 0))
   )
-  (wire (pts (xy 288.29 189.23) (xy 288.29 204.47))
+  (wire (pts (xy 288.29 189.23) (xy 288.29 200.66))
     (stroke (width 0) (type default) (color 0 0 0 0))
   )
@@
     (stroke (width 0) (type default) (color 0 0 0 0))
   )
+  (wire (pts (xy 312.42 200.66) (xy 312.42 207.01))
+    (stroke (width 0) (type default) (color 0 0 0 0))
+  )
   (wire (pts (xy 60.96 111.76) (xy 62.23 111.76))
     (stroke (width 0) (type default) (color 0 0 0 0))
@@
     (stroke (width 0) (type default) (color 0 0 0 0))
   )
+  (wire (pts (xy 288.29 200.66) (xy 288.29 204.47))
+    (stroke (width 0) (type default) (color 0 0 0 0))
+  )
+  (wire (pts (xy 327.66 90.17) (xy 327.66 86.36))
+    (stroke (width 0) (type default) (color 0 0 0 0))
+  )
   (wire (pts (xy 247.65 125.73) (xy 247.65 138.43))
     (stroke (width 0) (type default) (color 0 0 0 0))
@@
     (stroke (width 0) (type default) (color 0 0 0 0))
   )
+  (wire (pts (xy 312.42 207.01) (xy 320.04 207.01))
+    (stroke (width 0) (type default) (color 0 0 0 0))
+  )
   (wire (pts (xy 83.82 189.23) (xy 87.63 189.23))
     (stroke (width 0) (type default) (color 0 0 0 0))
@@
     (stroke (width 0) (type default) (color 0 0 0 0))
   )
+  (wire (pts (xy 303.53 90.17) (xy 303.53 111.76))
+    (stroke (width 0) (type default) (color 0 0 0 0))
+  )
   (wire (pts (xy 262.89 111.76) (xy 262.89 125.73))
     (stroke (width 0) (type default) (color 0 0 0 0))
@@
   )
   (wire (pts (xy 83.82 149.86) (xy 87.63 149.86))
+    (stroke (width 0) (type default) (color 0 0 0 0))
+  )
+  (wire (pts (xy 288.29 200.66) (xy 312.42 200.66))
     (stroke (width 0) (type default) (color 0 0 0 0))
   )
@@
     (pin "2")
   )
+  (symbol (lib_id "Connector:TestPoint") (at 320.04 207.01 0) (unit 1)
+    (in_bom yes) (on_board yes) (fields_autoplaced)
+    (property "Reference" "TP1" (id 0) (at 322.58 202.4379 0)
+      (effects (font (size 1.27 1.27)) (justify left))
+    )
+    (property "Value" "TestPoint" (id 1) (at 322.58 204.9779 0)
+      (effects (font (size 1.27 1.27)) (justify left))
+    )
+    (property "Footprint" "" (id 2) (at 325.12 207.01 0)
+      (effects (font (size 1.27 1.27)) hide)
+    )
+    (property "Datasheet" "~" (id 3) (at 325.12 207.01 0)
+      (effects (font (size 1.27 1.27)) hide)
+    )
+    (pin "1")
+  )
   (symbol (lib_id "2835 LED SMD:JB2835BWT-G-H40EA0000-N0000001") (at 87.63 138.43 0) (unit 1)
     (in_bom yes) (on_board yes) (fields_autoplaced)
@@
     (pin "1")
   )
+  (symbol (lib_id "Connector:TestPoint") (at 327.66 86.36 0) (unit 1)
+    (in_bom yes) (on_board yes) (fields_autoplaced)
+    (property "Reference" "TP2" (id 0) (at 330.2 81.7879 0)
+      (effects (font (size 1.27 1.27)) (justify left))
+    )
+    (property "Value" "" (id 1) (at 330.2 84.3279 0)
+      (effects (font (size 1.27 1.27)) (justify left))
+    )
+    (property "Footprint" "" (id 2) (at 332.74 86.36 0)
+      (effects (font (size 1.27 1.27)) hide)
+    )
+    (property "Datasheet" "~" (id 3) (at 332.74 86.36 0)
+      (effects (font (size 1.27 1.27)) hide)
+    )
+    (pin "1")
+  )
   (symbol (lib_id "power:GND") (at 125.73 204.47 0) (unit 1)
     (in_bom yes) (on_board yes) (fields_autoplaced)
@@
       (reference "LED49") (unit 1) (value "JB2835BWT-G-H40EA0000-N0000001") (footprint "2835-library:JB2835BWTGH40EA0000N0000001")
     )
-  )
+    (path "/7a6c7535-50d8-40a2-b546-4877a3982c75"
+      (reference "TP1") (unit 1) (value "TestPoint") (footprint "TestPoint:TestPoint_Pad_D3.0mm")
+    )
+    (path "/e6afcdd3-ddae-4a78-909e-bd793b740929"
+      (reference "TP2") (unit 1) (value "TestPoint") (footprint "TestPoint:TestPoint_Pad_D3.0mm")
+    )
+  )

Commit message: REV 3 with fab out
Other:
- note added: "49 LED PANEL"
- note added: "7 parallel 7 series"
- title: (none) -> 49 pcs LED PANEL
- moved on the sheet: LED1, LED10, LED11, LED12, LED13, LED14, LED15, LED16, LED17, LED18, LED19, LED2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

Commit message: RECTIFIED CONNECTION
Parts:
- TP1: footprint (none) -> TestPoint:TestPoint_Pad_D3.0mm
- TP2: value (none) -> TestPoint; footprint (none) -> TestPoint:TestPoint_Pad_D3.0mm
Connections:
- net +24V: no longer LED10.2, LED11.2, LED12.2, LED13.2, LED14.2, LED16.2, LED17.2, LED18.2, LED19.2, LED2.2, LED20.2, LED21.2, LED23.2, LED24.2, LED25.2, LED26.2, LED27.2, LED28.2, LED3.2, LED30.2, LED31.2, LED32.2, LED33.2, LED34.2, LED35.2, LED37.2, LED38.2, LED39.2, LED4.2, LED40.2, LED41.2, LED42.2, LED44.2, LED45.2, LED46.2, LED47.2, LED48.2, LED49.2, LED5.2, LED6.2, LED7.2, LED9.2
- net GND: no longer LED1.1, LED10.1, LED11.1, LED12.1, LED13.1, LED15.1, LED16.1, LED17.1, LED18.1, LED19.1, LED2.1, LED20.1, LED22.1, LED23.1, LED24.1, LED25.1, LED26.1, LED27.1, LED29.1, LED3.1, LED30.1, LED31.1, LED32.1, LED33.1, LED34.1, LED36.1, LED37.1, LED38.1, LED39.1, LED4.1, LED40.1, LED41.1, LED43.1, LED44.1, LED45.1, LED46.1, LED47.1, LED48.1, LED5.1, LED6.1, LED8.1, LED9.1
- new net: LED26.1, LED27.1
- new net: LED25.2, LED26.2
- new net: LED1.1, LED2.2
- new net: LED38.1, LED39.1
- new net: LED37.2, LED38.2
- new net: LED2.1, LED3.2
- new net: LED17.1, LED18.1
- new net: LED18.2, LED19.2
- new net: LED31.1, LED32.1
- new net: LED32.2, LED33.2
- new net: LED8.1, LED9.1
- new net: LED10.2, LED9.2
- new net: LED45.1, LED46.1
- new net: LED44.2, LED45.2
- new net: LED29.1, LED30.1
- new net: LED30.2, LED31.2
- new net: LED13.2, LED14.2
- new net: LED48.2, LED49.2
- new net: LED12.1, LED13.1
- new net: LED11.2, LED12.2
- new net: LED19.1, LED20.1
- new net: LED20.2, LED21.2
- new net: LED34.2, LED35.2
- new net: LED5.1, LED6.2
- new net: LED4.1, LED5.2
- new net: LED24.1, LED25.1
- new net: LED23.2, LED24.2
- new net: LED15.1, LED16.1
- new net: LED16.2, LED17.2
- new net: LED6.1, LED7.2
- new net: LED36.1, LED37.1
- new net: LED22.1, LED23.1
- new net: LED10.1, LED11.1
- new net: LED43.1, LED44.1
- new net: LED47.1, LED48.1
- new net: LED46.2, LED47.2
- new net: LED3.1, LED4.2
- new net: LED27.2, LED28.2
- new net: LED41.2, LED42.2
- new net: LED39.2, LED40.2
- new net: LED33.1, LED34.1
- new net: LED40.1, LED41.1
